Commit message: Updated CARMA URDF for Sensors

File: example_calibration_folder/vehicle/calibration/urdf/carma.urdf (robot description, URDF)
Before this commit: robot vehicle_platform, 13 links, 12 joints
Joints:
- removed joint mobileye
- removed joint radar_fc
- removed joint radar_fl
- removed joint radar_fr
- removed joint radar_rl
- removed joint radar_rr
- joint base_link_to_host_vehicle: origin xyz=3.37 0 -0.3556 rpy=3.14159265359 0 0 -> xyz=0.0523875 0 -0.06985 rpy=3.14159265359 0 0
- joint base_link_to_vehicle_front: origin xyz=4 0 0.57 rpy=0 0 0 -> xyz=0.2206625 0 0.06985 rpy=0 0 0
- joint lidar: origin xyz=1.02 0 2.23 rpy=0 0 0 -> xyz=0.1016 0 0 0.02195 rpy=0 0 0

Commit message: Example dev calibration folder for carla integration

File: example_calibration_folder/vehicle/calibration/urdf/carma.urdf (robot description, URDF)
Before this commit: robot vehicle_platform, 13 links, 12 joints
Links:
- removed link novatel_gnss
- added link gps
Joints:
- joint base_link_to_novatel: child novatel_gnss -> gps
- joint gnss_to_ned_heading: parent novatel_gnss -> gps

Commit message: fix urdf dimention

File: example_calibration_folder/vehicle/calibration/urdf/carma.urdf (robot description, URDF)
Before this commit: robot vehicle_platform, 13 links, 12 joints
Joints:
- joint base_link_to_vehicle_front: origin xyz=4 0 0.57 rpy=0 0 0 -> xyz=2.25 0 0.57 rpy=0 0 0

Commit message: Example dev calibration folder for carla integration (#345)
<!-- Thanks for the contribution, this is awesome. -->

# PR Details
## Description
When updating documentation at
https://usdot-carma.atlassian.net/wiki/spaces/CRMSIM/pages/2419916803/Setup+Instructions+Documentation+CARMA-CARLA+integration
Vehicle calibration folder needed to be updated for carma vehicles to
engage and run on carma-system-4.5.0.

This version is pulled straight from the most recent development
calibration on vehicle-calibration private repo, but needs to be updated
here for public access.
<!--- Describe your changes in detail -->

## Related Issue
https://usdot-carma.atlassian.net/browse/CXC-26

<!--- This project only accepts pull requests related to open issues -->
<!--- If suggesting a new feature or change, please discuss it in an
issue first -->
<!--- If fixing a bug, there should be an issue describing it with steps
to reproduce -->
<!--- Please link to the issue here: -->

## Motivation and Context
See above.
<!--- Why is this change required? What problem does it solve? -->

## How Has This Been Tested?
SIM PC 1 integration tested
<!--- Please describe in detail how you tested your changes. -->
<!--- Include details of your testing environment, and the tests you ran
to -->
<!--- see how your change affects other areas of the code, etc. -->

## Types of changes

<!--- What types of changes does your code introduce? Put an `x` in all
the boxes that apply: -->

- [ ] Defect fix (non-breaking change that fixes an issue)
- [X] New feature (non-breaking change that adds functionality)
- [ ] Breaking change (fix or feature that cause existing functionality
to change)

## Checklist:

<!--- Go over all the following points, and put an `x` in all the boxes
that apply. -->
<!--- If you're unsure about any of these, don't hesitate to ask. We're
here to help! -->

- [X] I have added any new packages to the sonar-scanner.properties file
- [X] My change requires a change to the documentation.
- [X] I have updated the documentation accordingly.
- [X] I have read the **CONTRIBUTING** document.
[CARMA Contributing
Guide](https://github.com/usdot-fhwa-stol/carma-platform/blob/develop/Contributing.md)
- [X] I have added tests to cover my changes.
- [X] All new and existing tests passed.

File: example_calibration_folder/vehicle/calibration/urdf/carma.urdf (robot description, URDF)
Before this commit: robot vehicle_platform, 13 links, 12 joints
Links:
- removed link novatel_gnss
- added link gps
Joints:
- joint base_link_to_novatel: child novatel_gnss -> gps
- joint base_link_to_vehicle_front: origin xyz=4 0 0.57 rpy=0 0 0 -> xyz=2.25 0 0.57 rpy=0 0 0
- joint gnss_to_ned_heading: parent novatel_gnss -> gps

Commit message: correct-urdf-for-carla-vehicle

File: example_calibration_folder/vehicle/calibration/urdf/carma.urdf (robot description, URDF)
Before this commit: robot vehicle_platform, 13 links, 12 joints
Joints:
- joint radar_fc: origin xyz=4 0 0.57 rpy=0 0 0 -> xyz=2.25 0 0.57 rpy=0 0 0

Commit message: add lexus

File: example_calibration_folder/vehicle/calibration/urdf/carma.urdf (robot description, URDF)
Before this commit: robot vehicle_platform, 13 links, 12 joints
Links:
- link base_link: geometry visual mesh filename=file:///opt/carma/vehicle/calibration/visualization_meshes/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 scale=0.001 0.001 0.001
